File: T41-2_Power.kicad_sch (KiCad schematic)
At the start: 34 parts, among them J1 Conn_02x08_Odd_Even, J2 Screw_Terminal_01x02, J3 Screw_Terminal_01x02, J4 Screw_Terminal_01x02, U1 R-78CK3.3-0.5, U2 R-78CK5.0-0.5

Commit message: Updated PDF schematic.
Other:
- note added: "5V OUT FOR DISPLAY"
Changed lines of the file:
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@@
 	(title_block
 		(title "T41-2 Power Supply")
-		(date "2024-04-02")
+		(date "2024-05-11")
+		(rev "V1.0")
 		(company "Greg KF5N")
 	)
@@
 			)
 		)
+	)
+	(text "5V OUT FOR DISPLAY"
+		(exclude_from_sim no)
+		(at 248.285 151.765 0)
+		(effects
+			(font
+				(size 2 2)
+				(thickness 0.4)
+				(bold yes)
+			)
+		)

Commit message: Updated schematic with note on V10/V11 versus T41-2 speaker connection.
Other:
- note added: "The speaker is routed for V10/V11 only! Do not place E7, E8, C16, C17, and J2 for use with the T41-2 Main Board."
