File: T41-2_Power.kicad_sch (KiCad schematic)
At the start: 34 parts, among them J1 Conn_02x08_Odd_Even, J2 Screw_Terminal_01x02, J3 Screw_Terminal_01x02, J4 Screw_Terminal_01x02, U1 R-78CK3.3-0.5, U2 R-78CK5.0-0.5

Commit message: Ready for fab V1.1.
Parts:
- removed C17: 0.1uf, Capacitor_SMD:C_1206_3216Metric, symbol Device:C_Small
- removed E8: 28F0121-0SR-10, 28F0121_0SR_10:FB_28F0121-0SR-10, symbol LairdFerrBead:28F0121-0SR-10
Connections:
- net 12V_SAFE: now also E7.2
- net GND: now also J2.2 (Pin_2)
- net at J2.1 (Pin_1): now also C16.2, E7.1
- net at J1.3 (Pin_3): no longer E7.2
- no-connect marks 2 -> 4
Other:
- note added: "+12V AUDIO AMP"
- note added: "5V OUT"
- note removed: "5V OUT FOR DISPLAY"
- note removed: "SPEAKER"
- note removed: "The speaker is routed for V10/V11 only! Do not place E7, E8, C16, C17, and J2 for use with the T41-2 Main Board."
- moved on the sheet: J2
