File: T41-2_Power.kicad_pcb (KiCad board)
At the start: 2 copper layers, 70 x 64 mm, 34 parts, among them J1 Conn_02x08_Odd_Even, J2 Screw_Terminal_01x02, J3 Screw_Terminal_01x02, J4 Screw_Terminal_01x02, U1 R-78CK3.3-0.5, U2 R-78CK5.0-0.5

Commit message: Ready for fab V1.1.
Parts:
- removed C17: 0.1uf, Capacitor_SMD:C_1206_3216Metric
- removed E8: 28F0121-0SR-10, 28F0121_0SR_10:FB_28F0121-0SR-10
- E7: moved to F.Cu
- moved E7 9.26 mm to (121.8, 70.5), turned to 0 degrees
- moved C7 2.75 mm to (134.0, 91.2)
- moved C16 2.56 mm to (116.3, 72.0), turned to 90 degrees
Connections:
- C16 pad 2: Net-(J2-Pin_2) -> Net-(J2-Pin_1)
- E7 pad 1: Net-(J2-Pin_2) -> Net-(J2-Pin_1)
- E7 pad 2: Net-(J1-Pin_3) -> /12V_SAFE
- J1 pad 3: Net-(J1-Pin_3) -> unconnected-(J1-Pin_3-Pad3)
- J1 pad 4: Net-(J1-Pin_4) -> unconnected-(J1-Pin_4-Pad4)
- J2 pad 2: Net-(J2-Pin_2) -> GND
Routing:
- net Net-(J1-Pin_4): track 31.6 -> 0.00 mm
- net /12V_SAFE: track 49.7 -> 78.7 mm
- net Net-(J1-Pin_3): track 26.7 -> 0.00 mm
- net Net-(J2-Pin_2): track 17.3 -> 0.00 mm
- net Net-(J2-Pin_1): track 22.1 -> 13.8 mm
- net GND: track 0.07 -> 0.12 mm, vias 53 -> 62
Other:
- board text added: "+5V SUPPLY"
- board text added: "12V AUDIO AMP"
- board text added: "V1.1"
- board text removed: "+5V DISPLAY"
- board text removed: "SPEAKER"
- board text removed: "V1.0"
